File: Robot/Robot.sch (KiCad schematic (older format))
At the start: 2 parts

Commit message: shema
shema
Parts:
- removed D?: LED, symbol LED
- removed R?: R, symbol R
- added Ard?: ArduinoMicro, symbol ArduinoMicro
- added BT?: BT, symbol BT
- added C? (x2): C, symbol C
- added EM1: Motor Levi, symbol Motor
- added EM2: Motor Desni, symbol Motor
- added L293?: L293, symbol L293
- added Mux?: Mux, symbol Mux
- added QR? (x8): QRE1113, symbol QRE1113
- added R?: 150R, symbol R
- added R? (x8): 10k, symbol R
Connections:
- net +5V: now also Ard?.29 (5V), BT?.1 (Vcc), EM1.3 (Vcc), EM2.3 (Vcc), L293?.1 (1,2EN), L293?.16 (Vcc1), L293?.9 (3,4EN), Mux?.16 (Vdd), R?.1, R?.1, R?.1, R?.1, R?.1, R?.1, R?.1, R?.1
- net GND: now also Ard?.31 (GND), Ard?.6 (GND), BT?.2 (GND), EM1.6 (GND), EM2.6 (GND), L293?.12 (GND), L293?.13 (GND), L293?.4 (GND), L293?.5 (GND), Mux?.6 (INH), Mux?.7 (Vee), Mux?.8 (Vss), QR?.4 (EM), QR?.4 (EM), QR?.4 (EM), QR?.4 (EM), QR?.4 (EM), QR?.4 (EM), QR?.4 (EM), QR?.4 (EM)
- new net: QR?.1 (A+), R?.2
- new net: QR?.1 (A+), QR?.2 (C-) (x7)
- new net: Mux?.13 (Ch_0), QR?.3 (COL), R?.2
- new net: Ard?.14 (9(PWM)/A9), L293?.10 (3A)
- new net: C?.2, EM2.2 (M2), L293?.11 (3Y)
- new net: C?.1, EM2.1 (M1), L293?.14 (4Y)
- new net: Ard?.15 (10(PWM)/A10), L293?.15 (4A)
- new net: Ard?.10 (5(PWM)), L293?.2 (1A)
- new net: C?.1, EM1.1 (M1), L293?.3 (1Y)
- new net: C?.2, EM1.2 (M2), L293?.6 (2Y)
- new net: Ard?.11 (6(PWM)), L293?.7 (2A)
- new net: Mux?.1 (Ch_4), QR?.3 (COL), R?.2
- new net: Ard?.13 (8/A8), Mux?.10 (B)
- new net: Ard?.12 (7), Mux?.11 (A)
- new net: Mux?.12 (Ch_3), QR?.3 (COL), R?.2
- new net: Mux?.14 (Ch_1), QR?.3 (COL), R?.2
- new net: Mux?.15 (Ch_2), QR?.3 (COL), R?.2
- new net: Mux?.2 (Ch_6), QR?.3 (COL), R?.2
- new net: Ard?.21 (A0), Mux?.3 (COM_O/I)
- new net: Mux?.4 (Ch_7), QR?.3 (COL), R?.2
- new net: Mux?.5 (Ch_5), QR?.3 (COL), R?.2
- new net: Ard?.17 (12/A11), Mux?.9 (C)
- new net: Ard?.3 (1/TX), BT?.4 (Rx_5V)
- new net: Ard?.4 (0/RX), BT?.3 (Tx_5V)
- new net +9V: Ard?.32 (VIN), L293?.8 (Vcc2), R?.1

Commit message: pdf
pdf
Parts:
- added BT?: Baterija, symbol Battery
- added C?: 22uF, symbol CP1
- added R? (x2): 10k, symbol R
- added SW?: Switch_inv, symbol Switch_inv
Connections:
- net +9V: now also R?.1, SW?.2
- net GND: now also BT?.2 (-), C?.2, R?.2, SW?.3
- net ENCLA: now reaches EM1.4 (OutA)
- net ENCLA: now also Ard?.7 (2/SDA)
- net ENCLB: now reaches EM1.5 (OutB)
- net ENCLB: now also Ard?.3 (1/TX)
- net at Ard?.22 (A1): now also BT?.4 (Rx_5V)
- net at Ard?.23 (A2): now also BT?.3 (Tx_5V)
- net VBAT: now reaches Ard?.26 (A5)
- net VBAT: now also R?.1, R?.2
- net ENCRB: now reaches Ard?.4 (0/RX)
- net ENCRB: now also EM2.5 (OutB); no longer BT?.3 (Tx_5V)
- net ENCRA: now reaches Ard?.8 (3(PWM)/SCL)
- net ENCRA: now also EM2.4 (OutA)
- new net +9VA: BT?.1 (+), C?.1, SW?.1
Changed lines of the file:
@@
 EESchema Schematic File Version 2
+LIBS:Komponente
 LIBS:power
 LIBS:device
@@
 LIBS:contrib
 LIBS:valves
-LIBS:Komponente
 LIBS:Robot-cache
 EELAYER 25 0
@@
 	8950 5300 9100 5300
 Wire Wire Line
-	9100 5300 9100 5650
-Wire Wire Line
-	9100 5650 6200 5650
-Wire Wire Line
-	6200 5650 6200 4050
-Wire Wire Line
-	6200 4050 6300 4050
+	9100 5300 9100 5850
 Wire Wire Line
 	8950 5400 9050 5400
 Wire Wire Line
 	9050 5400 9050 5800
-Wire Wire Line
-	9050 5800 6150 5800
-Wire Wire Line
-	6150 5800 6150 3950
-Wire Wire Line
-	6150 3950 6300 3950
 $Comp
 L Motor EM2
@@
 Wire Wire Line
 	5600 5150 6300 5150
+Wire Wire Line
+	8150 2450 8250 2450
+Wire Wire Line
+	8250 2450 8250 3050
+Wire Wire Line
+	8250 3050 7950 3050
+Text GLabel 7950 3050 0    60   Input ~ 0
+ENCLA
+Wire Wire Line
+	6300 4350 5600 4350
+Text GLabel 5600 4350 0    60   Input ~ 0
+ENCLA
+Text GLabel 5600 4500 0    60   Input ~ 0
+ENCRA
+Wire Wire Line
+	6300 4450 5650 4450
+Wire Wire Line
+	5650 4450 5650 4500
+Wire Wire Line
+	5650 4500 5600 4500
+Wire Wire Line
+	10350 2500 10300 2500
+Wire Wire Line
+	10300 2500 10300 3100
+Text GLabel 10300 3100 3    60   Input ~ 0
+ENCRA
+Wire Wire Line
+	8150 2550 8150 3200
+Text GLabel 8150 3200 3    60   Input ~ 0
+ENCLB
+Wire Wire Line
+	10350 2600 10200 2600
+Wire Wire Line
+	10200 2600 10200 3550
+Text GLabel 10200 3550 3    60   Input ~ 0
+ENCRB
+Text GLabel 5450 3950 0    60   Input ~ 0
+ENCLB
+Text GLabel 5400 4150 0    60   Input ~ 0
+ENCRB
+Wire Wire Line
+	5400 4150 6050 4150
+Wire Wire Line
+	6050 4150 6050 4050
+Wire Wire Line
+	6050 4050 6300 4050
+Wire Wire Line
+	5450 3950 6300 3950
+Wire Wire Line
+	9050 5800 8200 5800
+Wire Wire Line
+	8200 5800 8200 4950
+Wire Wire Line
+	8200 4950 7500 4950
+Wire Wire Line
+	9100 5850 8050 5850
+Wire Wire Line
+	8050 5850 8050 4850
+Wire Wire Line
+	8050 4850 7500 4850
+$Comp
+L Battery BT?
+U 1 1 58C63780
+P 3450 6550
+F 0 "BT?" H 3550 6650 50  0000 L CNN
+F 1 "Baterija" H 3550 6550 50  0000 L CNN
+F 2 "" V 3450 6610 50  0000 C CNN
+F 3 "" V 3450 6610 50  0000 C CNN
+	1    3450 6550
+	1    0    0    -1
+$EndComp
+$Comp
+L +9VA #PWR?
+U 1 1 58C63E84
+P 3450 6150
+F 0 "#PWR?" H 3450 6025 50  0001 C CNN
+F 1 "+9VA" H 3450 6300 50  0000 C CNN
+F 2 "" H 3450 6150 50  0000 C CNN
+F 3 "" H 3450 6150 50  0000 C CNN
+	1    3450 6150
+	1    0    0    -1
+$EndComp
+Wire Wire Line
+	3450 6150 3450 6350
+Wire Wire Line
+	3450 6300 4750 6300
+Wire Wire Line
+	4100 6300 4100 6400
+Connection ~ 3450 6300
+$Comp
+L CP1 C?
+U 1 1 58C643A3
+P 4100 6550
+F 0 "C?" H 4125 6650 50  0000 L CNN
+F 1 "22uF" H 4125 6450 50  0000 L CNN
+F 2 "" H 4100 6550 50  0000 C CNN
+F 3 "" H 4100 6550 50  0000 C CNN
+	1    4100 6550
+	1    0    0    -1
+$EndComp
+Wire Wire Line
+	3450 6750 3450 6900
+Wire Wire Line
+	3450 6900 4750 6900
+Wire Wire Line
+	4100 6700 4100 6900
+Connection ~ 4100 6900
+Wire Wire Line
+	4400 6900 4400 7050
+Connection ~ 4400 6900
+$Comp
+L GND #PWR?
+U 1 1 58C64D0F
+P 4400 7050
+F 0 "#PWR?" H 4400 6800 50  0001 C CNN
+F 1 "GND" H 4400 6900 50  0000 C CNN
+F 2 "" H 4400 7050 50  0000 C CNN
+F 3 "" H 4400 7050 50  0000 C CNN
+	1    4400 7050
+	1    0    0    -1
+$EndComp
+$Comp
+L Switch_inv SW?
+U 1 1 58C6553D
+P 5150 6750
+F 0 "SW?" H 5300 6950 60  0000 C CNN
+F 1 "Switch_inv" H 5400 6600 60  0000 C CNN
+F 2 "" H 5150 6750 60  0001 C CNN
+F 3 "" H 5150 6750 60  0001 C CNN
+	1    5150 6750
+	1    0    0    -1
+$EndComp
+Wire Wire Line
+	4750 6300 4750 6600
+Connection ~ 4100 6300
+Wire Wire Line
+	5550 6750 5950 6750
+$Comp
+L +9V #PWR?
+U 1 1 58C66D44
+P 5950 6600
+F 0 "#PWR?" H 5950 6450 50  0001 C CNN
+F 1 "+9V" H 5950 6740 50  0000 C CNN
+F 2 "" H 5950 6600 50  0000 C CNN
+F 3 "" H 5950 6600 50  0000 C CNN
+	1    5950 6600
+	1    0    0    -1
+$EndComp
+Connection ~ 5950 6750
+$Comp
+L R R?
+U 1 1 58C66FBD
+P 5950 7000
+F 0 "R?" V 6030 7000 50  0000 C CNN
+F 1 "10k" V 5950 7000 50  0000 C CNN
+F 2 "" V 5880 7000 50  0000 C CNN
+F 3 "" H 5950 7000 50  0000 C CNN
+	1    5950 7000
+	1    0    0    -1
+$EndComp
+$Comp
+L R R?
+U 1 1 58C67BD4
+P 5950 7400
+F 0 "R?" V 6050 7400 50  0000 C CNN
+F 1 "10k" V 5950 7400 50  0000 C CNN
+F 2 "" V 5880 7400 50  0000 C CNN
+F 3 "" H 5950 7400 50  0000 C CNN
+	1    5950 7400
+	1    0    0    -1
+$EndComp
+Wire Wire Line
+	5950 6600 5950 6850
+Wire Wire Line
+	5950 7150 5950 7250
+Wire Wire Line
+	5950 7550 5950 7600
+$Comp
+L GND #PWR?
+U 1 1 58C6886B
+P 5950 7600
+F 0 "#PWR?" H 5950 7350 50  0001 C CNN
+F 1 "GND" H 5950 7450 50  0000 C CNN
+F 2 "" H 5950 7600 50  0000 C CNN
+F 3 "" H 5950 7600 50  0000 C CNN
+	1    5950 7600
+	1    0    0    -1
+$EndComp
+Wire Wire Line
+	5950 7200 5550 7200
+Connection ~ 5950 7200
+Text GLabel 5550 7200 0    60   Input ~ 0
+VBAT
+Text GLabel 7650 4550 2    60   Input ~ 0
+VBAT
+Wire Wire Line
+	7650 4550 7500 4550
 $EndSCHEMATC

Commit message: footprinti
Parts:
- gave numbers to parts that had none: 28

Commit message: pcb
Parts:
- removed C1: 22uF, symbol CP1
- added C1: C, Robot:C_0805_HandSoldering, symbol C
- Ard1: footprint (none) -> Robot:ARDUINO_MICRO_SHIELD
- BT1: footprint (none) -> Robot:Battery_holder_1291
- BT2: footprint (none) -> Robot:BT_Smirf
- C2, C3: footprint (none) -> Robot:C_0805_HandSoldering
- EM1, EM2: footprint (none) -> Robot:EM_holder
- L2931: footprint (none) -> Robot:L293
- Mux1: footprint (none) -> Robot:Mux_8Ch
- QR1, QR2, QR3, QR4, QR5, QR6, QR7, QR8: footprint (none) -> Robot:QRE1113GR
- R1, R10, R11, R2, R3, R4, R5, R6, R7, R8, R9: footprint (none) -> Robot:R_0805_HandSoldering
- SW1: footprint (none) -> Robot:Switch
Connections:
- net +9VA: now also C1.1
- net GND: now also C1.2
